File: Eagle Files/Freaq.brd (EAGLE design)
At the start: 73.9 x 106.4 mm, 30 parts, among them M1 ARDUINO-NANO-3.0

Commit message: updated Gerber File
Connections:
- net GND: now also C5.-
Changed lines of the file:
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@@
 <contactref element="PWR" pad="5"/>
 <contactref element="PWR" pad="8"/>
+<contactref element="C5" pad="-"/>
 </signal>
 <signal name="+5V">
